File: Bank.sch (KiCad schematic (older format))
At the start: 3 parts

Commit message: more
Parts:
- U3, U4: renamed from U?; footprint (none) -> stdpads:TSSOP-20_4.4x6.5mm_P0.65mm
- U5: renamed from U?; footprint (none) -> stdpads:TSSOP-16_4.4x5mm_P0.65mm
Connections:
- net B0: now also U3.12 (Q4); no longer U4.19 (Q7)
- net B1: now also U3.15 (Q5); no longer U4.16 (Q6)
- net B2: now also U3.16 (Q6); no longer U4.15 (Q5)
- net B3: now also U3.19 (Q7); no longer U4.12 (Q4)
- net B4: now also U3.2 (Q0); no longer U4.9 (Q3)
- net B5: now also U3.5 (Q1); no longer U4.6 (Q2)
- net B6: now also U3.6 (Q2); no longer U4.5 (Q1)
- net B7: now also U3.9 (Q3); no longer U4.2 (Q0)
- net D0: now also U3.13 (D4); no longer U3.18 (D7)
- net D1: now also U3.14 (D5); no longer U3.17 (D6)
- net D2: now also U3.17 (D6); no longer U3.14 (D5)
- net D3: now also U3.18 (D7); no longer U3.13 (D4)
- net D4: now also U3.3 (D0); no longer U3.8 (D3)
- net D5: now also U3.4 (D1); no longer U3.7 (D2)
- net D6: now also U3.7 (D2); no longer U3.4 (D1)
- net D7: now also U3.8 (D3); no longer U3.3 (D0)
- net W0: now also U4.19 (Q7); no longer U3.19 (Q7)
- net W1: now also U4.16 (Q6); no longer U3.16 (Q6)
- net W2: now also U4.15 (Q5); no longer U3.15 (Q5)
- net W3: now also U4.12 (Q4); no longer U3.12 (Q4)
- net W4: now also U4.9 (Q3); no longer U3.9 (Q3)
- net W5: now also U4.6 (Q2); no longer U3.6 (Q2)
- net W6d: now also U4.5 (Q1); no longer U3.5 (Q1)
- net W7d: now also U4.2 (Q0); no longer U3.2 (Q0)
- net BankSel renamed PHI2
- net ~BankSel~ renamed ~IO2~
- net ~WE~ renamed R~W~
