File: Control.sch (KiCad schematic (older format))
At the start: 6 parts, among them U12 74LVC02, U13 74LVC32, U14 74LVC00, U15 74LVC02, U16 74LVC32, U17 74LVC00

Commit message: PAL
Parts:
- removed U12, U15: 74LVC02, stdpads:TSSOP-14_4.4x5mm_P0.65mm, symbol 74xx:74LS02
- removed U13, U16: 74LVC32, stdpads:TSSOP-14_4.4x5mm_P0.65mm, symbol 74xx:74LS32
- removed U14, U17: 74LVC00, stdpads:TSSOP-14_4.4x5mm_P0.65mm, symbol 74xx:74LS00
- added R4: 47, stdpads:R_0603, symbol Device:R_Small
- added U11, U12: 74LVC273, stdpads:TSSOP-20_4.4x6.5mm_P0.65mm, symbol GW_Logic:74273
- added U13: 74AHC245PW, stdpads:TSSOP-20_4.4x6.5mm_P0.65mm, symbol GW_Logic:74245
- added U2: ATF16V8BQL, stdpads:PLCC-20_SMDSocket, symbol Logic_Programmable:GAL16V8
- added U9: 74LVC02, stdpads:TSSOP-14_4.4x5mm_P0.65mm, symbol 74xx:74LS02
Connections:
- net labels added: +3V3, +5V, DotClk, GND, PHI2, PHI2r1, PHI2r2, PHI2r3, RDQM_5, RSTr1, RSTr2, RSTr3, RSTr4, RSTr5, RSTr6, RSTr7, RSTr8, R~CAS~_5, R~CS~_5, R~RAS~_5, R~WE~_5, ~RST~
- net labels removed: Always, PHI2e3, PHI2e4, PHI2e5, PHI2e7, PHI2e8, RDWR, Ref0, Ref1, Ref8, ~RD~, ~WR~
- wire segments 557 -> 494
- no-connect marks 0 -> 8
Other:
- note added: "Command (preinit)"
- note added: "PHI2r1"
- note added: "PHI2r2"
- note added: "PHI2r3"
- note added: "R~RAS~ (idle)"
- note added: "R~RAS~ (read)"
- note added: "R~RAS~ (write)"
- note removed: "PHI0"
- note removed: "PHI02r1"
- note removed: "PHI02r2"
- note removed: "R~CS~ (idle)"
- note removed: "R~CS~ (read)"
- note removed: "R~CS~ (write)"
- note removed: "R~RAS~ (idle/read/write)"
