File: GW4301.sch (KiCad schematic (older format))
At the start: 37 parts, among them J1 C64, J2 JTAG, U1 M5LV-PQFP100, U2 DRAM_2Mx8, U3 LD1117S33

Commit message: idk
Parts:
- removed C14: 10p, stdpads:C_0805, symbol Device:C_Small
- removed J2: JTAG, Connector:Tag-Connect_TC2050-IDC-NL_2x05_P1.27mm_Vertical, symbol Connector_Generic:Conn_02x05_Odd_Even
- removed JP1: Mode, Connector_PinHeader_2.54mm:PinHeader_1x02_P2.54mm_Vertical_SMD_Pin1Left, symbol Device:Jumper_NO_Small
- removed JP2: Size, Connector_PinHeader_2.54mm:PinHeader_2x02_P2.54mm_Vertical_SMD, symbol Connector_Generic:Conn_02x02_Odd_Even
- removed R1, R2: 0, stdpads:R_0805, symbol Device:R_Small
- removed R3: 1k, stdpads:R_0805, symbol Device:R_Small
- removed R4: 470, stdpads:R_0805, symbol Device:R_Small
- removed R5, R6, R7, R8, R9: 22k, stdpads:R_0805, symbol Device:R_Small
- removed U1: M5LV-PQFP100, stdpads:PQFP-100_14x20mm_P0.65mm, symbol GW_PLD:M5LV-PQFP-100
- removed U2: DRAM_2Mx8, stdpads:SOJ-28-300mil, symbol GW_RAM:DRAM-2Mx8-SOP-28
- added U? (x2): 74AHCT00, symbol 74xx:74LS00
- added U?: MAX811LEUS-T, Package_TO_SOT_SMD:SOT-143, symbol Power_Supervisor:MAX811LEUS-T
- added U? (x3): 74LVC74PW, symbol 74xx:74LS74
- added U? (x2): 74LVC257, symbol GW_Logic:74257
- added U? (x2): 74LS02, symbol 74xx:74LS32
- added U?: W9864G6KH, stdpads:Winbond_TSOPII-54, symbol GW_RAM:SDRAM-16Mx16-TSOP2-54
Connections:
- net +3V3: now also C10.1, C11.1, C12.1, C13.1, U?.1 (VDD), U?.1 (~R), U?.10 (~S), U?.13 (~R), U?.14 (VDD), U?.15 (DQML), U?.16 (VCC), U?.16 (VCC), U?.27 (VDD), U?.3 (VDDQ), U?.3 (~MR), U?.37 (CKE), U?.4 (VCC), U?.4 (~S), U?.4 (~S), U?.43 (VDDQ), U?.49 (VDDQ), U?.9 (VDDQ)
- net +5V: no longer C10.1, C11.1, C12.1, C13.1
- net A0: now also U?.13 (D1)
- net A1: now also U?.10 (C1)
- net A2: now also U?.6 (B1)
- net A3: now also U?.3 (A1)
- net A4: now also U?.13 (D1)
- net A5: now also U?.10 (C1)
- net A6: now also U?.6 (B1)
- net A7: now also U?.3 (A1)
- net GND: now also U?.1 (GND), U?.12 (VSSQ), U?.15 (~OE~), U?.15 (~OE~), U?.28 (VSS), U?.36 (A12), U?.41 (VSS), U?.46 (VSSQ), U?.52 (VSSQ), U?.54 (VSS), U?.6 (VSSQ), U?.8 (GND), U?.8 (GND)
- net RA0: now also U?.12 (Zd), U?.23 (A0)
- net RA1: now also U?.24 (A1), U?.9 (Zc)
- net RA10: now also U?.22 (A10), U?.3
- net RA11: now also U?.35 (A11)
- net RA2: now also U?.25 (A2), U?.7 (Zb)
- net RA3: now also U?.26 (A3), U?.4 (Za)
- net RA4: now also U?.12 (Zd), U?.29 (A4)
- net RA5: now also U?.3, U?.30 (A5)
- net RA6: now also U?.31 (A6), U?.7 (Zb)
- net RA7: now also U?.32 (A7), U?.4 (Za)
- net RA8: now also U?.33 (A8)
- net RA9: now also U?.34 (A9)
- net RD0: now also U?.53 (DQ15)
- net RD1: now also U?.51 (DQ14)
- net RD2: now also U?.50 (DQ13)
- net RD3: now also U?.48 (DQ12)
- net RD4: now also U?.47 (DQ11)
- net RD5: now also U?.45 (DQ10)
- net RD6: now also U?.44 (DQ9)
- net RD7: now also U?.42 (DQ8)
- net R~WE~: now also U?.16 (~WE~)
- net R~W~: now also U?.2
- net ~IO1~: now also U?.1
- net ~IO2~: now also U?.2
- new net: U?.12 (D), U?.5 (Q)
- new net: U?.2 (D), U?.9 (Q)
- new net: U?.1, U?.9 (Zc)
- new net All: U?.2
- new net Amux: U?.1 (S), U?.1 (S)
- new net B0: U?.14 (D0)
- new net B1: U?.11 (C0)
- new net B2: U?.5 (B0)
- new net B3: U?.2 (A0)
- new net B4: U?.14 (D0)
- new net B5: U?.11 (C0)
- new net B6: U?.5 (B0)
- new net B7: U?.2 (A0)
- new net BODr: U?.6 (~Q)
- new net DotCk: U?.11 (C), U?.3 (C), U?.3 (C)
- new net ModeReg: U?.2
- new net RBA0: U?.20 (BA0)
- new net RBA1: U?.21 (BA1)
- new net RCLK: U?.38 (CLK)
- new net RDQM: U?.39 (DQMH)
- new net R~CAS~: U?.17 (~CAS~)
- new net R~CS~: U?.19 (~CS~)
- new net R~RAS~: U?.18 (~RAS~)
- new net US: U?.1, U?.3
- new net W2: U?.1
- new net ~BOD~: U?.1 (~R), U?.2 (D), U?.2 (~RESET)
- new net ~BOD~r: U?.5 (Q)
- no-connect marks 9 -> 10
Other:
- note added: "~A AND B~\n\n~A~ OR ~B~"
- moved on the sheet: C1, C10, C11, C12, C13, C2, C4, C5, C6, C7, C8, C9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

Commit message: more
Parts:
- removed U3: LD1117S33, stdpads:SOT-223, symbol Regulator_Linear:LD1117S33TR_SOT223
- removed U? (x2): 74AHCT00, symbol 74xx:74LS00
- removed U?: MAX811LEUS-T, Package_TO_SOT_SMD:SOT-143, symbol Power_Supervisor:MAX811LEUS-T
- removed U? (x3): 74LVC74PW, symbol 74xx:74LS74
- removed U? (x2): 74LVC257, symbol GW_Logic:74257
- removed U? (x2): 74LS02, symbol 74xx:74LS32
- removed U?: W9864G6KH, stdpads:Winbond_TSOPII-54, symbol GW_RAM:SDRAM-16Mx16-TSOP2-54
- added R2: 1k, stdpads:R_0603, symbol Device:R_Small
- added R3: 33, stdpads:R_0603, symbol Device:R_Small
- added U13: 74LVC32, stdpads:TSSOP-14_4.4x5mm_P0.65mm, symbol 74xx:74LS32
- added U19: XC6206P332MR, stdpads:SOT-23, symbol Regulator_Linear:XC6206PxxxMR
- C1, C2: footprint stdpads:C_0805 -> stdpads:C_0603
- C10: renamed from C11; footprint stdpads:C_0805 -> stdpads:C_0603
- C11: renamed from C12; footprint stdpads:C_0805 -> stdpads:C_0603
- C12: renamed from C13; footprint stdpads:C_0805 -> stdpads:C_0603
- C3: renamed from C4; footprint stdpads:C_0805 -> stdpads:C_0603
- C4: renamed from C5; footprint stdpads:C_0805 -> stdpads:C_0603
- C5: renamed from C6; footprint stdpads:C_0805 -> stdpads:C_0603
- C6: renamed from C7; footprint stdpads:C_0805 -> stdpads:C_0603
- C7: renamed from C8; footprint stdpads:C_0805 -> stdpads:C_0603
- C8: renamed from C9; footprint stdpads:C_0805 -> stdpads:C_0603
- C9: renamed from C10; footprint stdpads:C_0805 -> stdpads:C_0603
Connections:
- net +3V3: now also U19.2 (VO)
- net +5V: now also R2.1, U19.3 (VI)
- net DotClk: now also R2.2, U13.2
- net GND: now also U13.1, U19.1 (GND)
- net A10: no longer names the net of J1.34 (Pin_34)
- net A11: no longer names the net of J1.35 (Pin_35)
- net A12: no longer names the net of J1.36 (Pin_36)
- net A13: no longer names the net of J1.37 (Pin_37)
- net A14: no longer names the net of J1.38 (Pin_38)
- net A15: no longer names the net of J1.39 (Pin_39)
- net A8: no longer names the net of J1.32 (Pin_32)
- net A9: no longer names the net of J1.33 (Pin_33)
- net BA: no longer names the net of J1.12 (Pin_12)
- net ~DMA~: no longer names the net of J1.13 (Pin_13)
- net ~EXROM~: no longer names the net of J1.9 (Pin_9)
- net ~GAME~: no longer names the net of J1.8 (Pin_8)
- net ~IRQ~: no longer names the net of J1.4 (Pin_4)
- net ~NMI~: no longer names the net of J1.41 (Pin_41)
- net ~RESET~ renamed ~RST~
- net ~ROMH~: no longer names the net of J1.43 (Pin_43)
- net ~ROML~: no longer names the net of J1.11 (Pin_11)
- new net: R3.2, U13.3
- new net SDRAM/CLK: R3.1
- no-connect marks 10 -> 19
Other:
- note removed: "~A AND B~\n\n~A~ OR ~B~"
- moved on the sheet: C1, C10, C11, C12, C2, C3, C4, C5, C6, C7, C8, C9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

Commit message: PAL
Parts:
- removed U13: 74LVC32, stdpads:TSSOP-14_4.4x5mm_P0.65mm, symbol 74xx:74LS32
- added R1: 47, stdpads:R_0603, symbol Device:R_Small
- added U9: 74LVC02, stdpads:TSSOP-14_4.4x5mm_P0.65mm, symbol 74xx:74LS02
- R3: value 33 -> 47
Connections:
- net DotClk: now also U9.6
- net GND: now also U9.2, U9.5
- net SDRAM/CLK: now also R1.1, U9.3; no longer R3.1
- net at R3.2: now also U9.1
- new net: R1.2, U9.4
- new net Control/DotClk: R3.1
- no-connect marks 19 -> 16
Other:
- moved on the sheet: R2
