File: SDRAM.sch (KiCad schematic (older format))
At the start: 2 parts, among them U1 W9864G6KH, U2 74AHCT245PW

Commit message: PAL
Parts:
- U10: renamed from U2; value 74AHCT245PW -> 74AHC245PW
Changed lines of the file:
@@
 $Descr USLetter 11000 8500
 encoding utf-8
-Sheet 3 6
+Sheet 5 5
 Title ""
 Date ""
@@
 $EndComp
 $Comp
-L GW_Logic:74245 U2
+L GW_Logic:74245 U10
 U 1 1 61CAB158
 P 6400 3750
-F 0 "U2" H 6400 4350 50  0000 C CNN
-F 1 "74AHCT245PW" V 6400 3750 50  0000 C CNN
+F 0 "U10" H 6400 4350 50  0000 C CNN
+F 1 "74AHC245PW" V 6400 3750 50  0000 C CNN
 F 2 "stdpads:TSSOP-20_4.4x6.5mm_P0.65mm" H 6400 3100 50  0001 C TNN
 F 3 "" H 6400 3850 60  0001 C CNN
