File: State.sch (KiCad schematic (older format))
At the start: 8 parts

Commit message: more
Parts:
- removed U? (x3): 74LVC74PW, symbol 74xx:74LS74
- removed U?: 74LS02, symbol 74xx:74LS32
- removed U?: 74LS04, symbol 74xx:74LS04
- added C13: 2u2, stdpads:C_0603, symbol Device:C_Small
- added D1: 1N5819, stdpads:D_SOD-123, symbol Device:D_Schottky_Small_ALT
- added R1: 22k, stdpads:R_0603, symbol Device:R_Small
- added unit 2 of U12
- added unit 3 of U12
- added U8: LM555, stdpads:SOIC-8_3.9mm, symbol Timer:LM555
- added U9: 74LVC273, stdpads:TSSOP-20_4.4x6.5mm_P0.65mm, symbol GW_Logic:74273
- U10, U11: renamed from U?; footprint (none) -> stdpads:TSSOP-20_4.4x6.5mm_P0.65mm
- U12: renamed from U?; value 74LS02 -> 74LVC02; footprint (none) -> stdpads:TSSOP-14_4.4x5mm_P0.65mm
Connections:
- net labels added: +5V, DotClk, TR, ~BOD~, ~BOD~r0, ~RST~, ~RST~r, ~RST~r0
- net labels removed: DotCk
- wire segments 26 -> 166
- no-connect marks 0 -> 3
Other:
- note added: "DotCk (8 MHz)"
- note added: "PHI0"
- note added: "PHI2"
- note added: "PHI2 is registered twice to gain setup time for the gates U12A and U12B."
- note added: "PHI2e1"
- note added: "PHI2e2"
- note added: "PHI2e3"
- note added: "PHI2e3\n"
- note added: "PHI2e4"
- note added: "PHI2e5"
- note added: "PHI2e6"
- note added: "PHI2e7"
- note added: "PHI2e8"
- note added: "PHI2e[8..4] similar…"
- note added: "Ref[x+1]"
- note added: "Ref[x]"
- note added: "The PHI2e[8..1] signals are an eight-state one-hot state counter\nwhich counts out the eight 8 MHz dot clock cycles\ncomprising one 1 MHz PHI cycle.\nThese bits are reset by the POR pulse so that none of PHI2e[8..1]\nare high until power is good."
- note added: "The Ref[8…0] signals form another state counter which which is clocked\nat 1 MHz by the PHI1e8 state signal edge. The Ref[8…0] state counter\nwith all bits low and shifts a “1” into each successive bit at the beginning\nof each PHI1e8 state until all bits are high, where it remains until a power cycle."
- note added: "The power-on reset signal ~BOD~ is double-synchronized to create ~BOD~r\nso as to “make synchronous” the asynchronous reset of U10 and U11.\nThe C64 reset signal is also kept low when ~BOD~r is low,\nalthogh the POR time is ~~47ms, less than that of the C64, so the C64’s\nPOR pulse on the ~RST~ line is not nominally extended."
- note added: "These bits are a continuation of the one-hot state \ncounter shift register which begins in U10"
- note added: "U8 generates a reset pulse at power-on\nwhich is ultimately fed to U10 and U11."
- note added: "We also double-synchronize the C64’s reset signal\nbefore feeding it to the geoRAM registers."
- moved on the sheet: U10, U11, U12A

Commit message: PAL
Parts:
- removed C13: 2u2, stdpads:C_0603, symbol Device:C_Small
- removed D1: 1N5819, stdpads:D_SOD-123, symbol Device:D_Schottky_Small_ALT
- removed R1: 22k, stdpads:R_0603, symbol Device:R_Small
- removed U11: 74LVC273, stdpads:TSSOP-20_4.4x6.5mm_P0.65mm, symbol GW_Logic:74273
- removed unit 3 of U12
- removed U8: LM555, stdpads:SOIC-8_3.9mm, symbol Timer:LM555
Connections:
- net labels removed: +5V, PHI2r2, Ref0, Ref1, Ref2, Ref3, Ref4, Ref5, Ref6, Ref7, Ref8, TR, ~BOD~, ~BOD~r, ~BOD~r0
- wire segments 166 -> 65
- no-connect marks 3 -> 0
Other:
- note added: "PHI2r1"
- note removed: "PHI0"
- note removed: "PHI2e3\n"
- note removed: "PHI2e[8..4] similar…"
- note removed: "Ref[x+1]"
- note removed: "Ref[x]"
- note removed: "The Ref[8…0] signals form another state counter which which is clocked\nat 1 MHz by the PHI1e8 state signal edge. The Ref[8…0] state counter\nwith all bits low and shifts a “1” into each successive bit at the beginning\nof each PHI1e8 state until all bits are high, where it remains until a power cycle."
- note removed: "U8 generates a reset pulse at power-on\nwhich is ultimately fed to U10 and U11."
- moved on the sheet: U12A, U12B
